File: PCB/Proteus_Top.kicad_pcb (KiCad board)
At the start: 2 copper layers, 317.4 x 117.3 mm, 76 parts

Commit message: Mon Oct 16 12:56:28 PM BST 2023
Parts:
- removed the REF** at (343.3, 162.3)
- removed the REF** at (171.9, 162.3) (x2)
- removed the REF** at (67.1, 95.7)
- removed the REF** at (181.4, 133.8)
- removed the REF** at (352.9, 76.6)
- removed the REF** at (124.3, 133.8)
- removed the REF** at (133.8, 162.3)
- removed the REF** at (86.2, 76.6)
- removed the REF** at (314.8, 133.8)
- removed the REF** at (333.8, 133.8)
- removed the REF** at (162.4, 114.7)
- removed the REF** at (67.1, 76.6)
- removed the REF** at (257.6, 76.6)
- removed the REF** at (162.4, 133.8)
- removed the REF** at (105.2, 114.7)
- removed the REF** at (238.6, 114.7)
- removed the REF** at (143.3, 76.6)
- removed the REF** at (105.2, 95.7)
- removed the REF** at (181.4, 76.6)
- removed the REF** at (276.7, 114.7)
- removed the REF** at (238.6, 133.8)
- removed the REF** at (295.7, 95.7)
- removed the REF** at (76.6, 162.3)
- removed the REF** at (86.2, 95.7)
- removed the REF** at (86.2, 114.7)
- removed the REF** at (352.9, 133.8)
- removed the REF** at (286.2, 162.3)
- removed the REF** at (67.1, 133.8)
- removed the REF** at (314.8, 76.6)
- removed the REF** at (124.3, 76.6)
- removed the REF** at (333.8, 95.7)
- removed the REF** at (143.3, 114.7)
- removed the REF** at (181.4, 114.7)
- removed the REF** at (314.8, 114.7)
- removed the REF** at (124.3, 114.7)
- removed the REF** at (248.1, 162.3) (x2)
- removed the REF** at (257.6, 114.7)
- removed the REF** at (257.6, 95.7)
- removed the REF** at (333.8, 76.6)
- removed the REF** at (314.8, 95.7)
- removed the REF** at (295.7, 114.7)
- removed the REF** at (276.7, 95.7)
- removed the REF** at (95.7, 162.3)
- removed the REF** at (162.4, 95.7)
- removed the REF** at (257.6, 133.8)
- removed the REF** at (86.2, 133.8)
- removed the REF** at (124.3, 95.7)
- removed the REF** at (67.1, 114.7)
- removed the REF** at (295.7, 133.8)
- removed the REF** at (295.7, 76.6)
- removed the REF** at (305.2, 162.3)
- removed the REF** at (276.7, 76.6)
- removed the REF** at (352.9, 95.7)
- removed the REF** at (143.3, 133.8)
- removed the REF** at (324.3, 162.3)
- removed the REF** at (333.8, 114.7)
- removed the REF** at (162.4, 76.6)
- removed the REF** at (238.6, 95.7)
- removed the REF** at (352.9, 114.7)
- removed the REF** at (105.2, 133.8)
- removed the REF** at (105.2, 76.6)
- removed the REF** at (238.6, 76.6)
- removed the REF** at (143.3, 95.7)
- removed the REF** at (114.7, 162.3)
- removed the REF** at (181.4, 95.7)
- removed the REF** at (276.7, 133.8)
- added REF**: MX_FMask-with-cutout, Stencils:MX_FMask-with-cutout, F.Cu at (324.3, 162.3)
- added REF**: MX_FMask-with-cutout, Stencils:MX_FMask-with-cutout, F.Cu at (314.8, 114.7)
- added REF**: MX_FMask-with-cutout, Stencils:MX_FMask-with-cutout, F.Cu at (314.8, 95.7)
- added REF**: MX_FMask-with-cutout, Stencils:MX_FMask-with-cutout, F.Cu at (86.2, 76.6)
- added REF**: MX_FMask-with-cutout, Stencils:MX_FMask-with-cutout, F.Cu at (352.9, 114.7)
- added REF**: MX_FMask-with-cutout, Stencils:MX_FMask-with-cutout, F.Cu at (314.8, 76.6)
- added REF**: MX_FMask-with-cutout, Stencils:MX_FMask-with-cutout, F.Cu at (238.6, 76.6)
- added REF**: MX_FMask-with-cutout, Stencils:MX_FMask-with-cutout, F.Cu at (238.6, 95.7)
- added REF**: MX_FMask-with-cutout, Stencils:MX_FMask-with-cutout, F.Cu at (86.2, 95.7)
- added REF**: MX_FMask-with-cutout, Stencils:MX_FMask-with-cutout, F.Cu at (105.2, 95.7)
- added REF**: MX_FMask-with-cutout, Stencils:MX_FMask-with-cutout, F.Cu at (95.7, 162.3)
- added REF**: MX_FMask-with-cutout, Stencils:MX_FMask-with-cutout, F.Cu at (124.3, 76.6)
- added REF**: MX_FMask-with-cutout, Stencils:MX_FMask-with-cutout, F.Cu at (352.9, 133.8)
- added REF**: MX_FMask-with-cutout, Stencils:MX_FMask-with-cutout, F.Cu at (67.1, 114.7)
- added REF**: MX_FMask-with-cutout, Stencils:MX_FMask-with-cutout, F.Cu at (276.7, 133.8)
- added REF**: MX_FMask-with-cutout, Stencils:MX_FMask-with-cutout, F.Cu at (181.4, 76.6)
- added REF**: MX_FMask-with-cutout, Stencils:MX_FMask-with-cutout, F.Cu at (181.4, 114.7)
- added REF**: MX_FMask-with-cutout, Stencils:MX_FMask-with-cutout, F.Cu at (162.4, 114.7)
- added REF**: MX_FMask-with-cutout, Stencils:MX_FMask-with-cutout, F.Cu at (105.2, 114.7)
- added REF**: MX_FMask-with-cutout, Stencils:MX_FMask-with-cutout, F.Cu at (86.2, 133.8)
- added REF**: MX_FMask-with-cutout, Stencils:MX_FMask-with-cutout, F.Cu at (314.8, 133.8)
- added REF**: MX_FMask-with-cutout, Stencils:MX_FMask-with-cutout, F.Cu at (286.2, 162.3)
- added REF**: MX_FMask-with-cutout, Stencils:MX_FMask-with-cutout, F.Cu at (162.4, 133.8)
- added REF**: MX_FMask-with-cutout, Stencils:MX_FMask-with-cutout, F.Cu at (257.6, 114.7)
- added REF**: MX_FMask-with-cutout, Stencils:MX_FMask-with-cutout, F.Cu at (333.8, 114.7)
- added REF**: MX_FMask-with-cutout, Stencils:MX_FMask-with-cutout, F.Cu at (67.1, 95.7)
- added REF**: MX_FMask-with-cutout, Stencils:MX_FMask-with-cutout, F.Cu at (295.7, 76.6)
- added REF**: MX_FMask-with-cutout, Stencils:MX_FMask-with-cutout, F.Cu at (105.2, 133.8)
- added REF**: MX_FMask-with-cutout, Stencils:MX_FMask-with-cutout, F.Cu at (333.8, 133.8)
- added REF**: MX_FMask-with-cutout, Stencils:MX_FMask-with-cutout, F.Cu at (143.3, 76.6)
- added REF**: MX_FMask-with-cutout, Stencils:MX_FMask-with-cutout, F.Cu at (143.3, 95.7)
- added REF**: MX_FMask-with-cutout, Stencils:MX_FMask-with-cutout, F.Cu at (181.4, 133.8)
- added REF**: MX_FMask-with-cutout, Stencils:MX_FMask-with-cutout, F.Cu at (352.9, 76.6)
- added REF**: MX_FMask-with-cutout, Stencils:MX_FMask-with-cutout, F.Cu at (105.2, 76.6)
- added REF**: MX_FMask-with-cutout, Stencils:MX_FMask-with-cutout, F.Cu at (143.3, 133.8)
- added REF**: MX_FMask-with-cutout, Stencils:MX_FMask-with-cutout, F.Cu at (276.7, 114.7)
- added REF**: MX_FMask-with-cutout, Stencils:MX_FMask-with-cutout, F.Cu at (295.7, 133.8)
- added REF**: MX_FMask-with-cutout, Stencils:MX_FMask-with-cutout, F.Cu at (295.7, 114.7)
- added REF**: MX_FMask-with-cutout, Stencils:MX_FMask-with-cutout, F.Cu at (181.4, 95.7)
- added REF**: MX_FMask-with-cutout, Stencils:MX_FMask-with-cutout, F.Cu at (295.7, 95.7)
- added REF**: MX_FMask-with-cutout, Stencils:MX_FMask-with-cutout, F.Cu at (257.6, 133.8)
- added REF**: MX_FMask-with-cutout, Stencils:MX_FMask-with-cutout, F.Cu at (114.7, 162.3)
- added REF**: MX_FMask-with-cutout, Stencils:MX_FMask-with-cutout, F.Cu at (124.3, 133.8)
- added REF**: MX_FMask-with-cutout, Stencils:MX_FMask-with-cutout, F.Cu at (67.1, 133.8)
- added REF**: MX_FMask-with-cutout, Stencils:MX_FMask-with-cutout, F.Cu at (333.8, 76.6)
- added REF**: MX_FMask-with-cutout, Stencils:MX_FMask-with-cutout, F.Cu at (305.2, 162.3)
- added REF**: MX_FMask-with-cutout, Stencils:MX_FMask-with-cutout, F.Cu at (76.6, 162.3)
- added REF**: MX_FMask-with-cutout, Stencils:MX_FMask-with-cutout, F.Cu at (276.7, 76.6)
- added REF**: MX_FMask-with-cutout, Stencils:MX_FMask-with-cutout, F.Cu at (257.6, 76.6)
- added REF**: MX_FMask-with-cutout, Stencils:MX_FMask-with-cutout, F.Cu at (162.4, 76.6)
- added REF**: MX_FMask-with-cutout, Stencils:MX_FMask-with-cutout, F.Cu at (238.6, 133.8)
- added REF**: MX_FMask-with-cutout, Stencils:MX_FMask-with-cutout, F.Cu at (67.1, 76.6)
- added REF**: MX_FMask-with-cutout, Stencils:MX_FMask-with-cutout, F.Cu at (143.3, 114.7)
- added REF**: MX_FMask-with-cutout, Stencils:MX_FMask-with-cutout, F.Cu at (124.3, 95.7)
- added REF**: MX_FMask-with-cutout, Stencils:MX_FMask-with-cutout, F.Cu at (343.3, 162.3)
- added REF**: MX_FMask-with-cutout, Stencils:MX_FMask-with-cutout, F.Cu at (162.4, 95.7)
- added REF**: MX_FMask-with-cutout, Stencils:MX_FMask-with-cutout, F.Cu at (86.2, 114.7)
- added REF**: MX_FMask-with-cutout, Stencils:MX_FMask-with-cutout, F.Cu at (124.3, 114.7)
- added REF**: MX_FMask-with-cutout, Stencils:MX_FMask-with-cutout, F.Cu at (133.8, 162.3)
- added REF**: MX_FMask-with-cutout, Stencils:MX_FMask-with-cutout, F.Cu at (238.6, 114.7)
- added REF**: MX_FMask-with-cutout, Stencils:MX_FMask-with-cutout, F.Cu at (352.9, 95.7)
- added REF**: MX_FMask-with-cutout, Stencils:MX_FMask-with-cutout, F.Cu at (333.8, 95.7)
- added REF**: MX_FMask-with-cutout, Stencils:MX_FMask-with-cutout, F.Cu at (276.7, 95.7)
- added REF**: MX_FMask-with-cutout, Stencils:MX_FMask-with-cutout, F.Cu at (257.6, 95.7)
- added SW_2u-E6: MX, Stencils:Triple-Dual-2u-LED-stab-flip, F.Cu at (171.9, 162.3)
- added SW_2u-E6: MX, Stencils:Triple-Dual-2u-LED-stab-flip, F.Cu at (248.1, 162.3)
