File: PCB/Proteus_PCB.kicad_pcb (KiCad board)
At the start: 2 copper layers, 317.4 x 117.3 mm, 145 parts, among them J1 LED, K10 Blank, K11 Blank, K12 Blank, K13 Blank, K14 Blank, K15 Blank, K16 Blank, K17 Blank, K18 Blank, K19 Blank, K2 Blank, K20 Blank, K21 Blank, K22 Blank, K23 Blank, K24 Blank, K25 Blank, K26 Blank, K27 Blank, K28 Blank, K29 Blank, K3 Blank, K30 Blank, K31 Blank, K32 Blank, K33 Blank, K34 Blank, K35 Blank, K36 Blank, K37 Blank, K38 Blank, K39 Blank, K4 Blank, K40 Blank, K41 Blank, K42 Blank, K43 Blank, K44 Blank, K45 Blank, K46 Blank, K47 Blank, K48 Blank, K49 Blank, K5 Blank, K50 Blank, K51 Blank, K52 Blank, K53 Blank, K54 Blank, K55 Blank, K56 Blank, K57 Blank, K58 Blank, K59 Blank, K6 Blank, K60 Blank, K61 Blank, K62 Blank, K63 Blank, K64 Blank, K65 Blank, K7 Blank, K8 Blank, K9 Blank

Commit message: Mon Oct 23 02:52:20 PM BST 2023
Parts:
- renumbered K1 to K0, K2 to K1
Other:
- board text added: "PCB3D_BR_PROTEUS67"
- board text added: "PCB3D_TL_PROTEUS67"
Changed lines of the file:
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@@
     (property "ki_keywords" "switch normally-open pushbutton push-button")
     (attr through_hole)
-    (fp_text reference "K1" (at -2.54 -2.794) (layer "F.SilkS")
+    (fp_text reference "K0" (at -2.54 -2.794) (layer "F.SilkS")
         (effects (font (size 1 1) (thickness 0.15)))
     )
@@
     (property "ki_keywords" "switch normally-open pushbutton push-button")
     (attr through_hole)
-    (fp_text reference "K2" (at -2.54 -2.794) (layer "F.SilkS")
+    (fp_text reference "K1" (at -2.54 -2.794) (layer "F.SilkS")
         (effects (font (size 1 1) (thickness 0.15)))
     )
@@
   (gr_arc (start 359.22 154.705) (mid 359.963949 152.908949) (end 361.76 152.165)
     (stroke (width 0.05) (type default)) (layer "Edge.Cuts"))
+  (gr_text "PCB3D_BR_PROTEUS67" (at 375.9 183.25) (layer "F.SilkS")
+    (effects (font (size 1 1) (thickness 0.1)) (justify left bottom))
+  )
   (gr_text "Designed by: github.com/gzowski\nRevision: 1 (Non-Hotswap)" (at 356.325 175.175) (layer "F.SilkS")
     (effects (font (size 1 1) (thickness 0.1)) (justify right bottom))
   )
+  (gr_text "PCB3D_TL_PROTEUS67" (at 46.4 54.65) (layer "F.SilkS")
+    (effects (font (size 1 1) (thickness 0.1)) (justify left bottom))
+  )
   (segment (start 57.60254 71.09254) (end 57.6 71.09) (width 0.2) (layer "B.Cu") (net 1))
